Commit message: update

File: loco_manipulation_gym/resources/robots/airbot_piper/urdf/airbot_piper.urdf (robot description, URDF)
Before this commit: robot airbot, 17 links, 16 joints
Links:
- added link gripper_base, mass 0.45; collision mesh filename=../meshes/piper/gripper_base.STL; visual mesh filename=../meshes/piper/gripper_base.STL
- link arm_link00: mass 0.162352169522719 -> 1.02
- link arm_link01: mass 0.0978679932242825 -> 0.71
- link arm_link02: mass 0.289571136953082 -> 1.17
- link arm_link03: mass 0.290583247455324 -> 0.5
- link arm_link04: mass 0.127087348341362 -> 0.38
- link arm_link05: mass 0.144711209371719 -> 0.383
- link gripper_link: mass 0.150196458571266 -> 0.00699089613564366
- link gripper_link_left: mass 0.0264822490707451 -> 0.025
- link gripper_link_right: mass 0.0264822500394006 -> 0.025
Joints:
- added joint joint6_to_gripper_base: type fixed, parent gripper_link, child gripper_base, origin xyz=0 0 0 rpy=0 0 0
- joint arm_joint00: limit lower=-2.618 upper=2.618 effort=100 velocity=8.2 -> lower=-2.618 upper=2.168 effort=100 velocity=5; origin xyz=0 0 0.123 rpy=0 0 -1.5708 -> xyz=0 0 0.123 rpy=0 0 0
- joint arm_joint01: limit lower=0 upper=3.14 effort=100 velocity=8.2 -> lower=0 upper=3.14 effort=100 velocity=5; origin xyz=0 0 0 rpy=1.5708 -0.10095 -1.5708 -> xyz=0 0 0 rpy=1.5708 -0.1359 -3.1416
- joint arm_joint02: limit lower=-2.967 upper=0 effort=100 velocity=8.2 -> lower=-2.967 upper=0 effort=100 velocity=5; origin xyz=0.28503 0 0 rpy=0 0 1.3826 -> xyz=0.28503 0 0 rpy=0 0 -1.7939
- joint arm_joint03: axis 0 0 -1 -> 0 0 1; limit lower=-1.832 upper=1.832 effort=100 velocity=8.2 -> lower=-1.745 upper=1.745 effort=100 velocity=5; origin xyz=0.021984 0.25075 0 rpy=-1.5708 0 0 -> xyz=-0.021984 -0.25075 0 rpy=1.5708 0 0
- joint arm_joint04: limit lower=-1.22 upper=1.22 effort=100 velocity=8.2 -> lower=-1.22 upper=1.22 effort=100 velocity=5; origin xyz=0 0 0 rpy=1.5708 -0.087266 0 -> xyz=0 0 0 rpy=-1.5708 0 0
- joint arm_joint05: axis 0 0 -1 -> 0 0 1; limit lower=-3.14 upper=3.14 effort=100 velocity=8.2 -> lower=-2.0944 upper=2.0944 effort=100 velocity=3; origin xyz=0 0.091 0.0014165 rpy=-1.5708 -1.5708 0 -> xyz=8.8259E-05 -0.091 0 rpy=1.5708 0 0
- joint arm_joint06: axis 0 0 -1 -> 0 0 1; limit lower=0.0 upper=0.04 effort=100 velocity=1 -> lower=0 upper=0.035 effort=10 velocity=1; origin xyz=0 0 0.13503 rpy=1.5708 0 1.5708 -> xyz=0 0 0.1358 rpy=1.5708 0 0; parent gripper_link -> gripper_base
- joint arm_joint07: axis 0 0 1 -> 0 0 -1; limit lower=-0.04 upper=0.0 effort=100 velocity=1 -> lower=-0.035 upper=0 effort=10 velocity=1; origin xyz=0 0 0.13503 rpy=-1.5708 0 1.5708 -> xyz=0 0 0.1358 rpy=1.5708 0 -3.1416; parent gripper_link -> gripper_base
- joint trunk_arm_joint_base_0: origin xyz=0.018 0 0.072 rpy=0 0 0 -> xyz=0 0 0 rpy=0 0 0

File: loco_manipulation_gym/resources/robots/go2_piper/urdf/go2_piper.urdf (robot description, URDF)
Before this commit: robot go2_arx_description, 38 links, 37 joints
Links:
- added link gripper_base, mass 0.45; collision mesh filename=../meshes/piper/gripper_base.STL; visual mesh filename=../meshes/piper/gripper_base.STL
- link arm_link00: mass 0.162352169522719 -> 1.02
- link arm_link01: mass 0.0978679932242825 -> 0.71
- link arm_link02: mass 0.289571136953082 -> 1.17
- link arm_link03: mass 0.290583247455324 -> 0.5
- link arm_link04: mass 0.127087348341362 -> 0.38
- link arm_link05: mass 0.144711209371719 -> 0.383
- link gripper_link: mass 0.150196458571266 -> 0.00699089613564366
- link gripper_link_left: mass 0.0264822490707451 -> 0.025
- link gripper_link_right: mass 0.0264822500394006 -> 0.025
Joints:
- added joint joint6_to_gripper_base: type fixed, parent gripper_link, child gripper_base, origin xyz=0 0 0 rpy=0 0 0
- joint arm_joint00: limit lower=-2.618 upper=2.618 effort=100 velocity=2 -> lower=-2.618 upper=2.168 effort=100 velocity=5; origin xyz=0 0 0.123 rpy=0 0 -1.5708 -> xyz=0 0 0.123 rpy=0 0 0
- joint arm_joint01: limit lower=0 upper=3.14 effort=100 velocity=2 -> lower=0 upper=3.14 effort=100 velocity=5; origin xyz=0 0 0 rpy=1.5708 -0.10095 -1.5708 -> xyz=0 0 0 rpy=1.5708 -0.1359 -3.1416
- joint arm_joint02: limit lower=-2.967 upper=0 effort=100 velocity=2 -> lower=-2.967 upper=0 effort=100 velocity=5; origin xyz=0.28503 0 0 rpy=0 0 1.3826 -> xyz=0.28503 0 0 rpy=0 0 -1.7939
- joint arm_joint03: axis 0 0 -1 -> 0 0 1; limit lower=-1.832 upper=1.832 effort=100 velocity=2 -> lower=-1.745 upper=1.745 effort=100 velocity=5; origin xyz=0.021984 0.25075 0 rpy=-1.5708 0 0 -> xyz=-0.021984 -0.25075 0 rpy=1.5708 0 0
- joint arm_joint04: limit lower=-1.22 upper=1.22 effort=100 velocity=2 -> lower=-1.22 upper=1.22 effort=100 velocity=5; origin xyz=0 0 0 rpy=1.5708 -0.087266 0 -> xyz=0 0 0 rpy=-1.5708 0 0
- joint arm_joint05: axis 0 0 -1 -> 0 0 1; limit lower=-3.14 upper=3.14 effort=100 velocity=2 -> lower=-2.0944 upper=2.0944 effort=100 velocity=3; origin xyz=0 0.091 0.0014165 rpy=-1.5708 -1.5708 0 -> xyz=8.8259E-05 -0.091 0 rpy=1.5708 0 0
- joint arm_joint06: axis 0 0 -1 -> 0 0 1; limit lower=0.0 upper=0.04 effort=100 velocity=2 -> lower=0 upper=0.035 effort=10 velocity=1; origin xyz=0 0 0.13503 rpy=1.5708 0 1.5708 -> xyz=0 0 0.1358 rpy=1.5708 0 0; parent gripper_link -> gripper_base
- joint arm_joint07: axis 0 0 1 -> 0 0 -1; limit lower=-0.04 upper=0.0 effort=100 velocity=2 -> lower=-0.035 upper=0 effort=10 velocity=1; origin xyz=0 0 0.13503 rpy=-1.5708 0 1.5708 -> xyz=0 0 0.1358 rpy=1.5708 0 -3.1416; parent gripper_link -> gripper_base
